File: Mini_Drone.kicad_sch (KiCad schematic)
At the start: 45 parts, among them J1 Conn_01x02, J3 Conn_01x02, J4 Conn_01x06, Q1 AO3400A, Q2 AO3400A, Q3 AO3400A, Q4 AO3400A, SW2 Tactile Switch 3x4x2, SW3 Tactile Switch 3x4x2, U1 ESP32-S3-WROOM-1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

Commit message: sch completed need add net classes and route
Parts:
- added J7, J8: Conn_01x11, Connector_PinHeader_2.54mm:PinHeader_1x11_P2.54mm_Vertical, symbol Connector_Generic:Conn_01x11
- added R8, R9: 10k, Resistor_SMD:R_0201_0603Metric_Pad0.64x0.40mm_HandSolder, symbol Device:R
- added TP12, TP13, TP14, TP18, TP19, TP20, TP21, TP22, TP23, TP24, TP25, TP26, TP27, TP28, TP29: D0, TestPoint:TestPoint_Pad_D1.0mm, symbol Connector:TestPoint
- added TP15, TP16, TP17: GND, TestPoint:TestPoint_Pad_D1.0mm, symbol Connector:TestPoint
Connections:
- net D3 is gone; now on net M3: Q3.1 (G), R6.1
- net BAT+: now also TP22.1, TP23.1, TP24.1, TP25.1
- net GND: now also TP11.1, R8.1, R9.1, TP15.1, TP16.1, TP17.1, TP26.1, TP27.1, TP28.1, TP29.1
- net LED1: now also U1.6 (IO6), J8.1 (Pin_1); no longer U1.8 (IO15)
- net LED2: now also U1.7 (IO7), J8.2 (Pin_2); no longer U1.9 (IO16)
- net LED3: now also U1.8 (IO15), J8.3 (Pin_3); no longer U1.10 (IO17)
- net RX1: now also U1.11 (IO18); no longer U1.39 (IO1)
- net TX1: now also U1.10 (IO17); no longer U1.38 (IO2)
- net USB_D+: now also J8.6 (Pin_6)
- net USB_D-: now also J8.5 (Pin_5)
- net at C5.2, D6.2 (A), Q1.3 (D)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: no longer TP11.1
- net IO8: now reaches U1.12 (IO8)
- net IO8: now also J8.4 (Pin_4)
- net at U1.15 (IO3): now also R9.2
- net M3: now reaches U1.17 (IO9)
- net M3: now also TP13.1, TP19.1
- net IO10: now reaches U1.18 (IO10)
- net IO10: now also J8.7 (Pin_7)
- net IO11: now reaches U1.19 (IO11)
- net IO11: now also J8.8 (Pin_8)
- net IO12: now reaches U1.20 (IO12)
- net IO12: now also J8.9 (Pin_9)
- net IO13: now reaches U1.21 (IO13)
- net IO13: now also J8.10 (Pin_10)
- net IO14: now reaches U1.22 (IO14)
- net IO14: now also J7.1 (Pin_1)
- net IO21: now reaches U1.23 (IO21)
- net IO21: now also J7.2 (Pin_2)
- net IO47: now reaches U1.24 (IO47)
- net IO47: now also J7.3 (Pin_3)
- net IO48: now reaches U1.25 (IO48)
- net IO48: now also J7.4 (Pin_4)
- net at U1.26 (IO45): now also R8.2
- net IO35: now reaches U1.28 (IO35)
- net IO35: now also J7.5 (Pin_5)
- net IO36: now reaches U1.29 (IO36)
- net IO36: now also J7.6 (Pin_6)
- net IO37: now reaches U1.30 (IO37)
- net IO37: now also J7.7 (Pin_7)
- net IO38: now reaches U1.31 (IO38)
- net IO38: now also J7.8 (Pin_8)
- net IO39: now reaches U1.32 (IO39)
- net IO39: now also J7.9 (Pin_9)
- net IO49: now reaches U1.33 (IO40)
- net IO49: now also J7.10 (Pin_10)
- net IO41: now reaches U1.34 (IO41)
- net IO41: now also J7.11 (Pin_11)
- net IO42: now reaches U1.35 (IO42)
- net IO42: now also J8.11 (Pin_11)
- net D0 renamed M1
- net M1: now also U1.9 (IO16), TP18.1
- net D10 renamed M2
- net M2: now also U1.39 (IO1), TP12.1, TP20.1
- net D8 renamed M4
- net M4: now also U1.38 (IO2), TP14.1, TP21.1
Other:
- moved on the sheet: C1, C3, C5, C6, C7, D1, D2, D3, D4, D5, D6, D7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
